File: telakone.brd (EAGLE design)
At the start: 100 x 100 mm, 189 parts, among them X10 MPT0.5/8-2.54, X11 MPT0.5/8-2.54, X2 MPT0.5/8-2.54, X3 MPT0.5/8-2.54, X4 PIIKKIRIMA-2, X5 PIIKKIRIMA-5, X7 U.FL-R-SMT-1, X8 MPT0.5/8-2.54, X9 PIIKKIRIMA-3, Y1 PTH2.6-5.5SQ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

Commit message: update documentation
Parts:
- added U$11, U$13, U$15, U$3, U$5, U$7, U$9: DAFUG, dafug:DAFUG
Changed lines of the file:
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@@
 <element name="U$1" library="dafug" package="DAFUG" value="DAFUG" x="80.8" y="18.25" smashed="yes"/>
 <element name="Y5" library="EKE" package="PTH-2.6-5.5SQ" value="PTH2.6-5.5SQ" x="60" y="60"/>
+<element name="U$3" library="dafug" package="DAFUG" value="DAFUG" x="2.75" y="-3.3"/>
+<element name="U$5" library="dafug" package="DAFUG" value="DAFUG" x="2.75" y="-9.05"/>
+<element name="U$7" library="dafug" package="DAFUG" value="DAFUG" x="2.75" y="-14.8"/>
+<element name="U$9" library="dafug" package="DAFUG" value="DAFUG" x="2.75" y="-20.55"/>
+<element name="U$11" library="dafug" package="DAFUG" value="DAFUG" x="2.75" y="-26.3"/>
+<element name="U$13" library="dafug" package="DAFUG" value="DAFUG" x="2.75" y="-32.05"/>
+<element name="U$15" library="dafug" package="DAFUG" value="DAFUG" x="2.75" y="-37.8"/>
 </elements>
 <signals>

Commit message: update component values, add bom
Parts:
- C1, C37, C45: value (none) -> 220u 16V D
- C23, C24: value (none) -> 22p
- C32, C40, C53: value (none) -> 2u2 50V 0805
- C38, C47, C5, C50, C51, C7: value (none) -> 10n
- C4: value 10n 0603 -> 10n
- C46, C48, C49, C52, C56, C57: value (none) -> 100n
- C8, C9: value (none) -> 2u2
- R1: value 10k0 0603 -> 10k0
- R10, R11, R12, R13, R14, R15, R16, R19, R20, R21, R22, R23, R33, R34, R37, R38, R59, R6, R7, R8, R9: value (none) -> 2k00
- R17, R32, R43, R44, R5: value 1k -> 1k00
- R18, R24, R25, R42, R47, R50, R51: value (none) -> 499
- R2: value 5k90 0603 -> 5k90
- R31, R4: value 19k1 -> 19k1 1206
- R35: value 5k90 -> 5k90 1206
- R58: value 121 -> 121 1206
- V14, V25: value ESDAXXSC6 -> WURTH 82402304
- V16: value SMAJXXA -> SMAJ20A
- V21: value SMAJXXCA -> SMAJ20CA
- V27: value ESDAXXSC6 -> ESDA19SC6
